File: PITS/PITS.sch (KiCad schematic (older format))
At the start: 39 parts, among them M2 BME280, P1 CONN_02X20, P14 BATT, P2 BNC, P3 BNC, P4 BNC, P5 BNC, P6 Batt, P7 SENSOR, U1 HX1, U2 MAX-M8C/Q, U3 MTX2, U4 RFM9*, U7 MCP3426

Commit message: new Annotation and netlist
Parts:
- P1: renamed from P2; value BNC -> MWSL-1252
- P2: renamed from P3; value BNC -> APRS
- P3: renamed from P1; value CONN_02X20 -> GPIO
- P4: renamed from P5; value BNC -> LORA
- P7: renamed from P4; value BNC -> UKHAS
- P8: renamed from P14; value BATT -> 5V
- renumbered C14 to C1, C1 to C3, M2 to M1, P7 to P5, R8 to R10, R5 to R11, R7 to R12, R4 to R13, R2 to R14, R3 to R15, R14 to R2, R15 to R3, R20 to R4, R21 to R5, R22 to R6, R26 to R7, R24 to R8, R25 to R9, U4 to U3, U3 to U4, U7 to U5
Changed lines of the file:
@@
 $EndDescr
 $Comp
-L CONN_02X20 P1
+L CONN_02X20 P3
 U 1 1 58189273
 P 4750 4250
-F 0 "P1" H 4750 5300 50  0000 C CNN
-F 1 "CONN_02X20" V 4750 4250 50  0000 C CNN
+F 0 "P3" H 4750 5300 50  0000 C CNN
+F 1 "GPIO" V 4750 4250 50  0000 C CNN
 F 2 "Socket_Strips:Socket_Strip_Straight_2x20" H 4750 3300 50  0001 C CNN
 F 3 "" H 4750 3300 50  0000 C CNN
@@
 $EndComp
 $Comp
-L R R14
+L R R2
 U 1 1 581983DD
 P 1850 3200
-F 0 "R14" V 1930 3200 50  0000 C CNN
+F 0 "R2" V 1930 3200 50  0000 C CNN
 F 1 "330" V 1850 3200 50  0000 C CNN
 F 2 "Resistors_SMD:R_0603_HandSoldering" V 1780 3200 50  0001 C CNN
@@
 $EndComp
 $Comp
-L R R15
+L R R3
 U 1 1 58198843
 P 1850 3600
-F 0 "R15" V 1930 3600 50  0000 C CNN
+F 0 "R3" V 1930 3600 50  0000 C CNN
 F 1 "330" V 1850 3600 50  0000 C CNN
 F 2 "Resistors_SMD:R_0603_HandSoldering" V 1780 3600 50  0001 C CNN
@@
 $EndComp
 $Comp
-L R R20
+L R R4
 U 1 1 581988DE
 P 1850 4000
-F 0 "R20" V 1930 4000 50  0000 C CNN
+F 0 "R4" V 1930 4000 50  0000 C CNN
 F 1 "330" V 1850 4000 50  0000 C CNN
 F 2 "Resistors_SMD:R_0603_HandSoldering" V 1780 4000 50  0001 C CNN
@@
 $EndComp
 $Comp
-L R R21
+L R R5
 U 1 1 5819A3B0
 P 1850 4400
-F 0 "R21" V 1930 4400 50  0000 C CNN
+F 0 "R5" V 1930 4400 50  0000 C CNN
 F 1 "330" V 1850 4400 50  0000 C CNN
 F 2 "Resistors_SMD:R_0603_HandSoldering" V 1780 4400 50  0001 C CNN
@@
 $EndComp
 $Comp
-L R R22
+L R R6
 U 1 1 5819A3B7
 P 1850 4800
-F 0 "R22" V 1930 4800 50  0000 C CNN
+F 0 "R6" V 1930 4800 50  0000 C CNN
 F 1 "330" V 1850 4800 50  0000 C CNN
 F 2 "Resistors_SMD:R_0603_HandSoldering" V 1780 4800 50  0001 C CNN
@@
 LEDs
 $Comp
-L MCP3426 U7
+L MCP3426 U5
 U 1 1 581A77F7
 P 8800 4400
-F 0 "U7" H 9050 4750 60  0000 C CNN
+F 0 "U5" H 9050 4750 60  0000 C CNN
 F 1 "MCP3426" H 9025 3950 60  0000 C CNN
 F 2 "Housings_SOIC:SOIC-8_3.9x4.9mm_Pitch1.27mm" H 9200 5400 60  0001 C CNN
@@
 $EndComp
 $Comp
-L C C1
+L C C3
 U 1 1 581A7804
 P 8500 3550
-F 0 "C1" H 8525 3650 50  0000 L CNN
+F 0 "C3" H 8525 3650 50  0000 L CNN
 F 1 "100n" H 8525 3450 50  0000 L CNN
 F 2 "Capacitors_SMD:C_0603_HandSoldering" H 8538 3400 50  0001 C CNN
@@
 GPIO
 $Comp
-L RFM9* U4
+L RFM9* U3
 U 1 1 581B5A2A
 P 5800 1700
-F 0 "U4" H 5800 2450 60  0000 C CNN
+F 0 "U3" H 5800 2450 60  0000 C CNN
 F 1 "RFM9*" H 5800 950 60  0000 C CNN
 F 2 "RF_Modules:RFM9xW" H 5900 2900 60  0001 C CNN
@@
 $EndComp
 $Comp
-L BNC P5
+L BNC P4
 U 1 1 581B5A45
 P 5000 1600
-F 0 "P5" H 5010 1720 50  0000 C CNN
-F 1 "BNC" V 5110 1540 50  0000 C CNN
+F 0 "P4" H 5010 1720 50  0000 C CNN
+F 1 "LORA" V 5110 1540 50  0000 C CNN
 F 2 "Connectors:SMA_Edge_small" H 5000 1600 50  0001 C CNN
 F 3 "" H 5000 1600 50  0000 C CNN
@@
 LORA/RFM9*
 $Comp
-L MTX2 U3
+L MTX2 U4
 U 1 1 581BA550
 P 8800 1700
-F 0 "U3" H 9100 2050 60  0000 C CNN
+F 0 "U4" H 9100 2050 60  0000 C CNN
 F 1 "MTX2" H 9100 1350 60  0000 C CNN
 F 2 "RF_Modules:MTX2" H 9100 1300 60  0001 C CNN
@@
 NoConn ~ 9500 1900
 $Comp
-L R R2
+L R R14
 U 1 1 581BA565
 P 9700 1850
-F 0 "R2" V 9780 1850 50  0000 C CNN
+F 0 "R14" V 9780 1850 50  0000 C CNN
 F 1 "4k7" V 9700 1850 50  0000 C CNN
 F 2 "Resistors_SMD:R_0603_HandSoldering" V 9630 1850 50  0001 C CNN
@@
 $EndComp
 $Comp
-L R R4
+L R R13
 U 1 1 581BA56C
 P 9700 1250
-F 0 "R4" V 9780 1250 50  0000 C CNN
+F 0 "R13" V 9780 1250 50  0000 C CNN
 F 1 "4k7" V 9700 1250 50  0000 C CNN
 F 2 "Resistors_SMD:R_0603_HandSoldering" V 9630 1250 50  0001 C CNN
@@
 $EndComp
 $Comp
-L BNC P4
+L BNC P7
 U 1 1 581BA573
 P 7800 1600
-F 0 "P4" H 7810 1720 50  0000 C CNN
-F 1 "BNC" V 7910 1540 50  0000 C CNN
+F 0 "P7" H 7810 1720 50  0000 C CNN
+F 1 "UKHAS" V 7910 1540 50  0000 C CNN
 F 2 "Connectors:SMA_Edge_small" H 7800 1600 50  0001 C CNN
 F 3 "" H 7800 1600 50  0000 C CNN
@@
 $EndComp
 $Comp
-L BNC P3
+L BNC P2
 U 1 1 581BA58D
 P 900 6500
-F 0 "P3" H 910 6620 50  0000 C CNN
-F 1 "BNC" V 1010 6440 50  0000 C CNN
+F 0 "P2" H 910 6620 50  0000 C CNN
+F 1 "APRS" V 1010 6440 50  0000 C CNN
 F 2 "Connectors:SMA_Edge_small" H 900 6500 50  0001 C CNN
 F 3 "" H 900 6500 50  0000 C CNN
@@
 $EndComp
 $Comp
-L R R26
+L R R7
 U 1 1 581BA594
 P 2850 6600
-F 0 "R26" V 2930 6600 50  0000 C CNN
+F 0 "R7" V 2930 6600 50  0000 C CNN
 F 1 "20k" V 2850 6600 50  0000 C CNN
 F 2 "Resistors_SMD:R_0603_HandSoldering" V 2780 6600 50  0001 C CNN
@@
 $EndComp
 $Comp
-L R R3
+L R R15
 U 1 1 581BA5B3
 P 10050 1500
-F 0 "R3" V 10130 1500 50  0000 C CNN
+F 0 "R15" V 10130 1500 50  0000 C CNN
 F 1 "20k" V 10050 1500 50  0000 C CNN
 F 2 "Resistors_SMD:R_0603_HandSoldering" V 9980 1500 50  0001 C CNN
@@
 $EndComp
 $Comp
-L C_Small C14
+L C_Small C1
 U 1 1 581C4845
 P 2000 1950
-F 0 "C14" H 2010 2020 50  0000 L CNN
+F 0 "C1" H 2010 2020 50  0000 L CNN
 F 1 "100n" H 2010 1870 50  0000 L CNN
 F 2 "Capacitors_SMD:C_0603_HandSoldering" H 2000 1950 50  0001 C CNN
@@
 $EndComp
 $Comp
-L BNC P2
+L BNC P1
 U 1 1 581C4B0F
 P 900 1100
-F 0 "P2" H 910 1220 50  0000 C CNN
-F 1 "BNC" V 1010 1040 50  0000 C CNN
+F 0 "P1" H 910 1220 50  0000 C CNN
+F 1 "MWSL-1252" V 1010 1040 50  0000 C CNN
 F 2 "RF_Modules:MWSL1252" H 900 1100 50  0001 C CNN
 F 3 "" H 900 1100 50  0000 C CNN
@@
 GPS
 $Comp
-L R R8
+L R R10
 U 1 1 581E74D8
 P 5000 6350
-F 0 "R8" V 5080 6350 50  0000 C CNN
+F 0 "R10" V 5080 6350 50  0000 C CNN
 F 1 "4k7" V 5000 6350 50  0000 C CNN
 F 2 "Resistors_SMD:R_0603_HandSoldering" V 4930 6350 50  0001 C CNN
@@
 EXT-SENSORS
 $Comp
-L R R24
+L R R8
 U 1 1 581EB377
 P 4600 6350
-F 0 "R24" V 4680 6350 50  0000 C CNN
+F 0 "R8" V 4680 6350 50  0000 C CNN
 F 1 "4k7" V 4600 6350 50  0000 C CNN
 F 2 "Resistors_SMD:R_0603_HandSoldering" V 4530 6350 50  0001 C CNN
@@
 $EndComp
 $Comp
-L R R25
+L R R9
 U 1 1 581EB43F
 P 4800 6350
-F 0 "R25" V 4880 6350 50  0000 C CNN
+F 0 "R9" V 4880 6350 50  0000 C CNN
 F 1 "4k7" V 4800 6350 50  0000 C CNN
 F 2 "Resistors_SMD:R_0603_HandSoldering" V 4730 6350 50  0001 C CNN
@@
 $EndComp
 $Comp
-L CONN_01X02 P14
+L CONN_01X02 P8
 U 1 1 581F2693
 P 8900 6250
-F 0 "P14" H 8900 6400 50  0000 C CNN
-F 1 "BATT" V 9000 6250 50  0000 C CNN
+F 0 "P8" H 8900 6400 50  0000 C CNN
+F 1 "5V" V 9000 6250 50  0000 C CNN
 F 2 "Connectors:SMD_2_xsmall" H 8900 6250 50  0001 C CNN
 F 3 "" H 8900 6250 50  0000 C CNN
@@
 $EndComp
 $Comp
-L BME280 M2
+L BME280 M1
 U 1 1 585C19A3
 P 6800 6200
-F 0 "M2" H 6800 6450 60  0000 C CNN
+F 0 "M1" H 6800 6450 60  0000 C CNN
 F 1 "BME280" H 6800 5950 60  0000 C CNN
 F 2 "RF_Modules:BME280_edit" H 6800 5900 60  0001 C CNN
@@
 I_neg
 $Comp
-L CONN_01X05 P7
+L CONN_01X05 P5
 U 1 1 59A1C9F2
 P 5600 6700
-F 0 "P7" H 5600 7000 50  0000 C CNN
+F 0 "P5" H 5600 7000 50  0000 C CNN
 F 1 "SENSOR" V 5700 6700 50  0000 C CNN
 F 2 "Connectors:SMD_5_xsmall" H 5600 6700 50  0001 C CNN
@@
 L1 & R1:\nOnly necessary\nfor active Antenna
 $Comp
-L R R5
+L R R11
 U 1 1 5A0DD198
 P 7200 4350
-F 0 "R5" V 7280 4350 50  0000 C CNN
+F 0 "R11" V 7280 4350 50  0000 C CNN
 F 1 "15k" V 7200 4350 50  0000 C CNN
 F 2 "Resistors_SMD:R_0805_HandSoldering" V 7130 4350 50  0001 C CNN
@@
 $EndComp
 $Comp
-L R R7
+L R R12
 U 1 1 5A0DD501
 P 7200 4850
-F 0 "R7" V 7280 4850 50  0000 C CNN
+F 0 "R12" V 7280 4850 50  0000 C CNN
 F 1 "10k" V 7200 4850 50  0000 C CNN
 F 2 "Resistors_SMD:R_0805_HandSoldering" V 7130 4850 50  0001 C CNN

Commit message: fertiggit add Pinbelegung.ods !
Parts:
- M1: footprint RF_Modules:BME280_edit -> (none)
Changed lines of the file:
@@
 Sheet 1 2
 Title "UgoesSky-V3.0b-PITS"
-Date "2017-11-16"
-Rev "B"
+Date "2018-05-08"
+Rev "C"
 Comp "Jonas Gappert"
 Comment1 ""
@@
 F 0 "M1" H 6800 6450 60  0000 C CNN
 F 1 "BME280" H 6800 5950 60  0000 C CNN
-F 2 "RF_Modules:BME280_edit" H 6800 5900 60  0001 C CNN
+F 2 "" H 6800 5900 60  0001 C CNN
 F 3 "" H 6800 5900 60  0001 C CNN
 	1    6800 6200
