File: PITS/Power.sch (KiCad schematic (older format))
At the start: 5 parts, among them M1 TPS61030, Q1 Q_PMOS_DGS, Q2 Q_PNP_dual

Commit message: new Annotation and netlist
Parts:
- Q1: renamed from Q2; value Q_PNP_dual -> DMMT5401
- Q2: renamed from Q1; value Q_PMOS_DGS -> DMP1045U
- renumbered M1 to M2, R6 to R16, R19 to R17
Changed lines of the file:
@@
 $EndComp
 $Comp
-L Q_PMOS_DGS Q1
+L Q_PMOS_DGS Q2
 U 1 1 581E4244
 P 6900 3300
-F 0 "Q1" H 7200 3350 50  0000 R CNN
-F 1 "Q_PMOS_DGS" H 7550 3250 50  0000 R CNN
+F 0 "Q2" H 7200 3350 50  0000 R CNN
+F 1 "DMP1045U" H 7550 3250 50  0000 R CNN
 F 2 "TO_SOT_Packages_SMD:SOT-23_Handsoldering" H 7100 3400 50  0001 C CNN
 F 3 "" H 6900 3300 50  0000 C CNN
@@
 	7400 3900 7400 4100
 $Comp
-L R R6
+L R R16
 U 1 1 581E4257
 P 6400 4250
-F 0 "R6" V 6480 4250 50  0000 C CNN
+F 0 "R16" V 6480 4250 50  0000 C CNN
 F 1 "10k" V 6400 4250 50  0000 C CNN
 F 2 "Resistors_SMD:R_0603_HandSoldering" V 6330 4250 50  0001 C CNN
@@
 $EndComp
 $Comp
-L R R19
+L R R17
 U 1 1 581E425E
 P 7400 4250
-F 0 "R19" V 7480 4250 50  0000 C CNN
+F 0 "R17" V 7480 4250 50  0000 C CNN
 F 1 "47k" V 7400 4250 50  0000 C CNN
 F 2 "Resistors_SMD:R_0603_HandSoldering" V 7330 4250 50  0001 C CNN
@@
 $EndComp
 $Comp
-L Q_PNP_dual Q2
+L Q_PNP_dual Q1
 U 1 1 585C40A3
 P 6500 3700
-F 0 "Q2" H 6700 3750 50  0000 L CNN
-F 1 "Q_PNP_dual" H 6700 3650 50  0000 L CNN
+F 0 "Q1" H 6700 3750 50  0000 L CNN
+F 1 "DMMT5401" H 6700 3650 50  0000 L CNN
 F 2 "TO_SOT_Packages_SMD:SOT-23-6_Handsoldering" H 6700 3800 50  0001 C CNN
 F 3 "" H 6500 3700 50  0000 C CNN
@@
 $EndComp
 $Comp
-L Q_PNP_dual Q2
+L Q_PNP_dual Q1
 U 2 1 585C4126
 P 7300 3700
-F 0 "Q2" H 7500 3750 50  0000 L CNN
-F 1 "Q_PNP_dual" H 7500 3650 50  0000 L CNN
+F 0 "Q1" H 7500 3750 50  0000 L CNN
+F 1 "DMMT5401" H 7500 3650 50  0000 L CNN
 F 2 "TO_SOT_Packages_SMD:SOT-23-6_Handsoldering" H 7500 3800 50  0001 C CNN
 F 3 "" H 7300 3700 50  0000 C CNN
@@
 $EndComp
 $Comp
-L LM7805CT M1
+L LM7805CT M2
 U 1 1 598E0500
 P 4400 3250
-F 0 "M1" H 4200 3450 50  0000 C CNN
+F 0 "M2" H 4200 3450 50  0000 C CNN
 F 1 "TPS61030" H 4400 3450 50  0000 L CNN
 F 2 "power:TPS61030" H 4400 3350 50  0001 C CIN

Commit message: fertiggit add Pinbelegung.ods !
Parts:
- M2: footprint power:TPS61030 -> (none)
Changed lines of the file:
@@
 Sheet 2 2
 Title "UgoesSky-V3.0b-PITS"
-Date "2017-11-16"
-Rev "B"
+Date "2018-05-08"
+Rev "C"
 Comp "Jonas Gappert"
 Comment1 ""
@@
 F 0 "M2" H 4200 3450 50  0000 C CNN
 F 1 "TPS61030" H 4400 3450 50  0000 L CNN
-F 2 "power:TPS61030" H 4400 3350 50  0001 C CIN
+F 2 "" H 4400 3350 50  0001 C CIN
 F 3 "" H 4400 3250 50  0000 C CNN
 	1    4400 3250
